File: first-pcb.kicad_pcb (KiCad board)
At the start: 2 copper layers, 0 parts

Commit message: PCB Started
Parts:
- added C1: 0.1uF, Capacitor_SMD:C_0805_2012Metric, B.Cu at (57.0, 65.7)
- added C2: 0.1uF, Capacitor_SMD:C_0805_2012Metric, B.Cu at (69.7, 82.2)
- added C3: 22pF, Capacitor_SMD:C_0805_2012Metric, B.Cu at (71.4, 59.1)
- added C4: 22pF, Capacitor_SMD:C_0805_2012Metric, B.Cu at (60.5, 59.1)
- added C5: 0.1uF, Capacitor_SMD:C_0805_2012Metric, B.Cu at (75.3, 69.1)
- added C6: 10uF, Capacitor_SMD:C_0805_2012Metric, B.Cu at (62.2, 82.2)
- added C7: C_Small, Capacitor_SMD:C_0805_2012Metric, B.Cu at (56.9, 73.9)
- added D1: D_Small, Diode_SMD:D_SOD-123, B.Cu at (100.8, 64.3)
- added D2: D_Small, Diode_SMD:D_SOD-123, B.Cu at (119.9, 64.3)
- added D3: D_Small, Diode_SMD:D_SOD-123, B.Cu at (100.8, 83.3)
- added D4: D_Small, Diode_SMD:D_SOD-123, B.Cu at (119.9, 83.3)
- added F1: 500mA, Fuse:Fuse_1206_3216Metric, F.Cu at (160.2, 76.7)
- added MX1: MX-NoLED, MX_Alps_Hybrid:MX-1U-NoLED, F.Cu at (92.9, 64.3)
- added MX2: MX-NoLED, MX_Alps_Hybrid:MX-1U-NoLED, F.Cu at (111.9, 64.3)
- added MX3: MX-NoLED, MX_Alps_Hybrid:MX-1U-NoLED, F.Cu at (92.9, 83.3)
- added MX4: MX-NoLED, MX_Alps_Hybrid:MX-1U-NoLED, F.Cu at (111.9, 83.3)
- added R1: 22, Resistor_SMD:R_0805_2012Metric, F.Cu at (159.6, 84.3)
- added R2: 22, Resistor_SMD:R_0805_2012Metric, F.Cu at (184.3, 62.1)
- added R3: 10k, Resistor_SMD:R_0805_2012Metric, F.Cu at (173.6, 70.2)
- added R4: 10k, Resistor_SMD:R_0805_2012Metric, B.Cu at (75.3, 76.3)
- added SW1: SW_Push, random-keyboard-parts:SKQG-1155865, F.Cu at (162.2, 68.5)
- added U1: ATmega32U4-AU, Package_QFP:TQFP-44_10x10mm_P0.8mm, B.Cu at (66.0, 73.2)
- added USB1: Molex-0548190589, random-keyboard-parts:Molex-0548190589, F.Cu at (176.2, 56.1)
- added Y1: 16MHz, Crystal:Crystal_SMD_3225-4Pin_3.2x2.5mm, B.Cu at (65.9, 59.1)
